File: IMU7Click_Update/IMU7Click_ICM.kicad_sch (KiCad schematic)
At the start: 14 parts, among them IC1 ICM-42688-P, J1 Conn_01x08, J2 Conn_01x08, Q1 NMOS

Commit message: Started some tracing of routes. Had to add and remove everything because I fucked up
Parts:
- removed IC1: ICM-42688-P, IIM42352, symbol ICM-42688-P:ICM-42688-P
- removed J1, J2: Conn_01x08, symbol Connector_Generic:Conn_01x08
- removed JP1: SolderJumper_3_Bridged12, symbol Jumper:SolderJumper_3_Bridged12
- added JP1: SolderJumper_3_Open, Jumper:SolderJumper-3_P1.3mm_Open_RoundedPad1.0x1.5mm_NumberLabels, symbol Jumper:SolderJumper_3_Open
- added U1: ~, mikroBUS:MIKROBUS_HOST_CONN, symbol mikroBUS:mikroBUS_Module
- added U2: ICM-42688-P, ICM-42688-P:ICM-42688-P, symbol IMU_ICM:ICM-42688-P
- C1, C2, C3: footprint (none) -> Capacitor_SMD:C_0603_1608Metric_Pad1.08x0.95mm_HandSolder
- D1: footprint (none) -> LED_SMD:LED_0805_2012Metric_Pad1.15x1.40mm_HandSolder
- Q1: footprint (none) -> Package_TO_SOT_SMD:SOT-23-3
- R1, R2, R3, R4, R5: footprint (none) -> Resistor_SMD:R_0603_1608Metric_Pad0.98x0.95mm_HandSolder
Connections:
- net +3V3: now also JP1.1 (A), U1.P7 (+3V3), U2.12 (AP_CS), U2.5 (VDDIO), U2.8 (VDD)
- net GND: now also U1.P8 (GND), U1.P9 (GND)
- net GND1: now also JP1.3 (B), U2.11 (RESV), U2.6 (GND), U2.7 (RESV)
- net IMU_EN: now also U1.P3 (CS)
- net I2C_SCL: now reaches R4.2
- net I2C_SCL: now also U1.P12 (SCL), U2.13 (AP_SCL)
- net I2C_SDA: now reaches R5.2
- net I2C_SDA: now also U1.P11 (SDA), U2.14 (AP_SDA)
- net at R2.2: now also U1.P15 (INT1), U2.4 (INT1)
- net at R3.2: now also U1.P16 (PWM), U2.9 (INT2)
- new net: JP1.2 (C), U2.1 (AP_AD0)
- no-connect marks 11 -> 8
Other:
- company: (none) -> University of Cape Town
- title: (none) -> IMU7Click_ICM-42688-P
- moved on the sheet: C1, C2, C3, D1, Q1, R1, R2, R3, R4, R5
